Commit message: setup vehicle and sensor_kit

File: src/sensor_kit/vm_sensor_kit_launch/vm_sensor_kit_description/urdf/sensor_kit.xacro (robot description, xacro)
@@ -2,4 +2,6 @@
 <robot xmlns:xacro="http://ros.org/wiki/xacro">
   <xacro:macro name="sensor_kit_macro" params="*origin parent:=base_link">
+    <!-- include xacro file -->
+    <!-- define args -->
     <xacro:arg name="gpu" default="false"/>
     <xacro:arg name="config_dir" default="$(find vm_sensor_kit_description)/config"/>
@@ -16,5 +18,5 @@
     <xacro:property name="calibration" value="${xacro.load_yaml('$(arg config_dir)/sensor_kit_calibration.yaml')}"/>
     <link name="camera_front" />
-    <link name="camera_front_right" />
+    <link name="camera1" />
     <link name="gnss" />
     <link name="rs16_top_base_link" />
@@ -45,14 +47,14 @@
              ${calibration['sensor_kit_base_link']['camera_front']['yaw']}" />
     </joint>
-    <joint name="camera_front_right_joint" type="fixed">
+    <joint name="camera1_joint" type="fixed">
       <parent link="sensor_kit_base_link" />
-      <child link="camera_front_right" />
+      <child link="camera1" />
       <origin
-        xyz="${calibration['sensor_kit_base_link']['camera_front_right']['x']}
-             ${calibration['sensor_kit_base_link']['camera_front_right']['y']}
-             ${calibration['sensor_kit_base_link']['camera_front_right']['z']}"
-        rpy="${calibration['sensor_kit_base_link']['camera_front_right']['roll']}
-             ${calibration['sensor_kit_base_link']['camera_front_right']['pitch']}
-             ${calibration['sensor_kit_base_link']['camera_front_right']['yaw']}" />
+        xyz="${calibration['sensor_kit_base_link']['camera1']['x']}
+             ${calibration['sensor_kit_base_link']['camera1']['y']}
+             ${calibration['sensor_kit_base_link']['camera1']['z']}"
+        rpy="${calibration['sensor_kit_base_link']['camera1']['roll']}
+             ${calibration['sensor_kit_base_link']['camera1']['pitch']}
+             ${calibration['sensor_kit_base_link']['camera1']['yaw']}" />
     </joint>
     <!-- gnss -->

Commit message: feat localization

File: src/sensor_kit/vm_sensor_kit_launch/vm_sensor_kit_description/urdf/sensor_kit.xacro (robot description, xacro)
@@ -23,4 +23,5 @@
     <link name="front_radar" />
     <link name="rear_radar" />
+    <link name="imu_link" />
     <!-- lidar -->
     <joint name="rs16_top_base_link_joint" type="fixed">
@@ -71,4 +72,15 @@
     </joint>
     <!-- imu -->
+    <joint name="imu_link" type="fixed">
+      <parent link="sensor_kit_base_link" />
+      <child link="imu_link" />
+      <origin
+        xyz="${calibration['sensor_kit_base_link']['imu_link']['x']}
+             ${calibration['sensor_kit_base_link']['imu_link']['y']}
+             ${calibration['sensor_kit_base_link']['imu_link']['z']}"
+        rpy="${calibration['sensor_kit_base_link']['imu_link']['roll']}
+             ${calibration['sensor_kit_base_link']['imu_link']['pitch']}
+             ${calibration['sensor_kit_base_link']['imu_link']['yaw']}" />
+    </joint>
     <!-- millimeter wave radar -->
     <joint name="front_radar_joint" type="fixed">
